File: src/kicad/HelloHi.kicad_pcb (KiCad board)
At the start: 2 copper layers, 100 x 100 mm, 66 parts, among them J1 Conn_01x02, Q1 BCV29, Q2 BCV29, SW1 SW_Push, SW2 SW_Push

Commit message: Add files via upload
Parts:
- moved R1 25.9 mm to (166.2, 103.7)
- moved R2 25.9 mm to (179.2, 103.7)
- moved R3 25.9 mm to (172.2, 104.1)
- moved R4 25.9 mm to (191.6, 111.2)
- moved R6 25.9 mm to (202.1, 106.2)
- moved SW1 25.9 mm to (172.5, 121.5)
- moved SW2 25.9 mm to (185.0, 117.0)
- moved Q1 25.9 mm to (176.7, 96.7)
- moved Q2 25.9 mm to (184.0, 106.7)
- moved R5 25.9 mm to (186.4, 96.2)
- moved J1 25.9 mm to (202.2, 121.5)
Routing:
- net GND: track 546.8 -> 522.7 mm
- net VCC2: track 375.0 -> 351.0 mm
- net VCC1: track 196.8 -> 190.2 mm
Other:
- board size 100 x 100 mm -> 100 x 76.2 mm
